Commit message: checkpoint: preserve integrated Go2 exploration workspace

File: src/simulator/Utils/go2_description/xacro/const.xacro (robot description, xacro)
@@ -48,6 +48,12 @@
     <xacro:property name="calf_rotor_offset_z" value="0.0"/>
     <!-- joint limits -->
-    <xacro:property name="damping" value="0.0"/>
-    <xacro:property name="friction" value="0.0"/>
+    <!-- The trained deployment contract puts all damping in the policy's PD
+         loop (kd=1.0), so at damping="0.0" a fast transient has no passive
+         damping anywhere: the legs ring and a joint pins at its velocity
+         limit.  These are a robustness floor, not a match to the trained
+         plant: raise damping to test the insufficient-damping hypothesis, and
+         restore 0.0 / 0.0 to run the exact trained plant. -->
+    <xacro:property name="damping" value="0.5"/>
+    <xacro:property name="friction" value="0.05"/>
     <xacro:property name="hip_position_max" value="1.0472"/>
     <xacro:property name="hip_position_min" value="-1.0472"/>

File: src/simulator/Utils/go2_description/xacro/gazebo.xacro (robot description, xacro)
@@ -3,4 +3,6 @@
   <xacro:macro name="go2_foot_contact" params="leg">
     <gazebo reference="${leg}_foot">
+      <!-- Keep stand-up contact compliant enough to release small lateral
+           errors instead of turning them into large body impulses. -->
       <mu1>0.6</mu1>
       <mu2>0.6</mu2>
@@ -16,9 +18,23 @@
   </xacro:macro>
   <xacro:macro name="go2_gazebo">
+    <!-- The planning proxy is intentionally not a dynamics experiment.  Make
+         the canonical root kinematic so contact impulses and gravity cannot
+         accumulate roll / pitch while VelocityControl integrates x/y/yaw.
+         rl_effort leaves the link fully dynamic. -->
+    <xacro:if value="$(arg terrain_velocity_control)">
+      <gazebo reference="base">
+        <kinematic>true</kinematic>
+        <gravity>false</gravity>
+      </gazebo>
+    </xacro:if>
     <gazebo>
-      <plugin filename="libgz_ros2_control-system.so"
-              name="gz_ros2_control::GazeboSimROS2ControlPlugin">
-        <parameters>$(find go2_description)/config/ros2_controllers.yaml</parameters>
-      </plugin>
+      <!-- Locked legs leave no joint to control; loading gz_ros2_control would
+           only create a controller_manager with nothing to manage. -->
+      <xacro:unless value="$(arg lock_legs)">
+        <plugin filename="libgz_ros2_control-system.so"
+                name="gz_ros2_control::GazeboSimROS2ControlPlugin">
+          <parameters>$(find go2_description)/config/ros2_controllers.yaml</parameters>
+        </plugin>
+      </xacro:unless>
       <!-- Always publish odometry, regardless of control mode -->
       <plugin filename="ignition-gazebo-odometry-publisher-system"

File: src/simulator/Utils/go2_description/xacro/leg.xacro (robot description, xacro)
@@ -1,28 +1,30 @@
 <?xml version="1.0"?>
 <robot xmlns:xacro="http://www.ros.org/wiki/xacro">
-    <xacro:macro name="leg" params="name mirror mirror_dae front_hind front_hind_dae">
-        <joint name="${name}_hip_joint" type="revolute">
+    <xacro:macro name="leg" params="name mirror mirror_dae front_hind front_hind_dae lock_legs:=false hip_lock:=0.0 thigh_lock:=0.0 calf_lock:=0.0">
+        <joint name="${name}_hip_joint" type="${'fixed' if lock_legs else 'revolute'}">
             <xacro:if value="${(mirror_dae == False) and (front_hind_dae == True)}">
-                <origin rpy="0 0 0" xyz="${leg_offset_x} ${-leg_offset_y} 0"/>
+                <origin rpy="${hip_lock if lock_legs else 0} 0 0" xyz="${leg_offset_x} ${-leg_offset_y} 0"/>
             </xacro:if>
             <xacro:if value="${(mirror_dae == True) and (front_hind_dae == True)}">
-                <origin rpy="0 0 0" xyz="${leg_offset_x} ${leg_offset_y} 0"/>
+                <origin rpy="${hip_lock if lock_legs else 0} 0 0" xyz="${leg_offset_x} ${leg_offset_y} 0"/>
             </xacro:if>
             <xacro:if value="${(mirror_dae == False) and (front_hind_dae == False)}">
-                <origin rpy="0 0 0" xyz="${-leg_offset_x} ${-leg_offset_y} 0"/>
+                <origin rpy="${hip_lock if lock_legs else 0} 0 0" xyz="${-leg_offset_x} ${-leg_offset_y} 0"/>
             </xacro:if>
             <xacro:if value="${(mirror_dae == True) and (front_hind_dae == False)}">
-                <origin rpy="0 0 0" xyz="${-leg_offset_x} ${leg_offset_y} 0"/>
+                <origin rpy="${hip_lock if lock_legs else 0} 0 0" xyz="${-leg_offset_x} ${leg_offset_y} 0"/>
             </xacro:if>
             <parent link="trunk"/>
             <child link="${name}_hip"/>
-            <axis xyz="1 0 0"/>
-            <dynamics damping="${damping}" friction="${friction}"/>
-            <xacro:if value="${(mirror_dae == True)}">
-                <limit effort="${hip_torque_max}" velocity="${hip_velocity_max}" lower="${hip_position_min}" upper="${hip_position_max}"/>
-            </xacro:if>
-            <xacro:if value="${(mirror_dae == False)}">
-                <limit effort="${hip_torque_max}" velocity="${hip_velocity_max}" lower="${-hip_position_max}" upper="${-hip_position_min}"/>
-            </xacro:if>
+            <xacro:unless value="${lock_legs}">
+                <axis xyz="1 0 0"/>
+                <dynamics damping="${damping}" friction="${friction}"/>
+                <xacro:if value="${(mirror_dae == True)}">
+                    <limit effort="${hip_torque_max}" velocity="${hip_velocity_max}" lower="${hip_position_min}" upper="${hip_position_max}"/>
+                </xacro:if>
+                <xacro:if value="${(mirror_dae == False)}">
+                    <limit effort="${hip_torque_max}" velocity="${hip_velocity_max}" lower="${-hip_position_max}" upper="${-hip_position_min}"/>
+                </xacro:if>
+            </xacro:unless>
         </joint>
         <joint name="${name}_hip_rotor_joint" type="fixed">
@@ -61,5 +63,5 @@
                 <!-- <material name="orange"/> -->
             </visual>
-            <collision name="${name}_foot_collision">
+            <collision name="${name}_hip_collision">
                 <origin rpy="${PI/2.0} 0 0" xyz="0 ${hip_offset*mirror} 0"/>
                 <geometry>
@@ -99,11 +101,13 @@
             </inertial>
         </link>
-        <joint name="${name}_thigh_joint" type="revolute">
-            <origin rpy="0 0 0" xyz="0 ${thigh_offset*mirror} 0"/>
+        <joint name="${name}_thigh_joint" type="${'fixed' if lock_legs else 'revolute'}">
+            <origin rpy="0 ${thigh_lock if lock_legs else 0} 0" xyz="0 ${thigh_offset*mirror} 0"/>
             <parent link="${name}_hip"/>
             <child link="${name}_thigh"/>
-            <axis xyz="0 1 0"/>
-            <dynamics damping="${damping}" friction="${friction}"/>
-            <limit effort="${thigh_torque_max}" velocity="${thigh_velocity_max}" lower="${thigh_position_min}" upper="${thigh_position_max}"/>
+            <xacro:unless value="${lock_legs}">
+                <axis xyz="0 1 0"/>
+                <dynamics damping="${damping}" friction="${friction}"/>
+                <limit effort="${thigh_torque_max}" velocity="${thigh_velocity_max}" lower="${thigh_position_min}" upper="${thigh_position_max}"/>
+            </xacro:unless>
         </joint>
         <joint name="${name}_thigh_rotor_joint" type="fixed">
@@ -163,11 +167,13 @@
             </inertial>
         </link>
-        <joint name="${name}_calf_joint" type="revolute">
-            <origin rpy="0 0 0" xyz="0 0 ${-thigh_length}"/>
+        <joint name="${name}_calf_joint" type="${'fixed' if lock_legs else 'revolute'}">
+            <origin rpy="0 ${calf_lock if lock_legs else 0} 0" xyz="0 0 ${-thigh_length}"/>
             <parent link="${name}_thigh"/>
             <child link="${name}_calf"/>
-            <axis xyz="0 1 0"/>
-            <dynamics damping="${damping}" friction="${friction}"/>
-            <limit effort="${calf_torque_max}" velocity="${calf_velocity_max}" lower="${calf_position_min}" upper="${calf_position_max}"/>
+            <xacro:unless value="${lock_legs}">
+                <axis xyz="0 1 0"/>
+                <dynamics damping="${damping}" friction="${friction}"/>
+                <limit effort="${calf_torque_max}" velocity="${calf_velocity_max}" lower="${calf_position_min}" upper="${calf_position_max}"/>
+            </xacro:unless>
         </joint>
         <joint name="${name}_calf_rotor_joint" type="fixed">
@@ -235,5 +241,5 @@
                 <!-- <material name="orange"/> -->
             </visual>
-            <collision>
+            <collision name="${name}_foot_collision">
                 <origin rpy="0 0 0" xyz="0 0 0"/>
                 <geometry>

File: src/simulator/Utils/go2_description/xacro/robot.xacro (robot description, xacro)
@@ -4,4 +4,9 @@
     <xacro:arg name="use_gazebo" default="true"/>
     <xacro:arg name="terrain_velocity_control" default="false"/>
+    <!-- Lock the 12 leg joints at the nominal stance and drop every leg
+         controller.  Used by the kinematic proxy mode, where the trunk is held
+         rigidly at the spawn height by the model itself: leg dynamics must not
+         decide the body height, because the local map trusts the LiDAR pose. -->
+    <xacro:arg name="lock_legs" default="false"/>
     <xacro:include filename="$(find go2_description)/xacro/const.xacro"/>
     <xacro:include filename="$(find go2_description)/xacro/materials.xacro"/>
@@ -135,10 +140,20 @@
     </link>
 -->
-    <xacro:leg name="FR" mirror="-1" mirror_dae= "False" front_hind="1"  front_hind_dae="True"  />
-    <xacro:leg name="FL" mirror="1"  mirror_dae="True"   front_hind="1"  front_hind_dae="True"  />
-    <xacro:leg name="RR" mirror="-1" mirror_dae="False"  front_hind="-1" front_hind_dae="False" />
-    <xacro:leg name="RL" mirror="1"  mirror_dae="True"   front_hind="-1" front_hind_dae="False" />
+    <!-- Stance angles matching DEFAULT_DOF_POS in the locomotion supervisor:
+         hip 0.1 (mirrored per side), thigh 0.8 front / 1.0 rear, calf -1.5. -->
+    <xacro:leg name="FR" mirror="-1" mirror_dae= "False" front_hind="1"  front_hind_dae="True"
+               lock_legs="$(arg lock_legs)" hip_lock="${-0.1}" thigh_lock="0.8" calf_lock="-1.5" />
+    <xacro:leg name="FL" mirror="1"  mirror_dae="True"   front_hind="1"  front_hind_dae="True"
+               lock_legs="$(arg lock_legs)" hip_lock="${0.1}" thigh_lock="0.8" calf_lock="-1.5" />
+    <xacro:leg name="RR" mirror="-1" mirror_dae="False"  front_hind="-1" front_hind_dae="False"
+               lock_legs="$(arg lock_legs)" hip_lock="${-0.1}" thigh_lock="1.0" calf_lock="-1.5" />
+    <xacro:leg name="RL" mirror="1"  mirror_dae="True"   front_hind="-1" front_hind_dae="False"
+               lock_legs="$(arg lock_legs)" hip_lock="${0.1}" thigh_lock="1.0" calf_lock="-1.5" />
     <xacro:if value="$(arg use_gazebo)">
-        <xacro:go2_ros2_control/>
+        <!-- With fixed legs there is nothing for ros2_control to command, so no
+             hardware interface and no controller_manager are created. -->
+        <xacro:unless value="$(arg lock_legs)">
+            <xacro:go2_ros2_control/>
+        </xacro:unless>
         <xacro:go2_gazebo/>
     </xacro:if>

File: src/simulator/Utils/go2_description/xacro/ros2_control.xacro (robot description, xacro)
@@ -25,16 +25,16 @@
         <plugin>gz_ros2_control/GazeboSimSystem</plugin>
       </hardware>
-      <xacro:go2_control_joint name="FL_hip_joint"/>
-      <xacro:go2_control_joint name="FL_thigh_joint" initial="0.8"/>
-      <xacro:go2_control_joint name="FL_calf_joint" initial="-1.5"/>
-      <xacro:go2_control_joint name="FR_hip_joint"/>
-      <xacro:go2_control_joint name="FR_thigh_joint" initial="0.8"/>
-      <xacro:go2_control_joint name="FR_calf_joint" initial="-1.5"/>
-      <xacro:go2_control_joint name="RL_hip_joint"/>
-      <xacro:go2_control_joint name="RL_thigh_joint" initial="0.8"/>
-      <xacro:go2_control_joint name="RL_calf_joint" initial="-1.5"/>
-      <xacro:go2_control_joint name="RR_hip_joint"/>
-      <xacro:go2_control_joint name="RR_thigh_joint" initial="0.8"/>
-      <xacro:go2_control_joint name="RR_calf_joint" initial="-1.5"/>
+      <xacro:go2_control_joint name="FL_hip_joint" effort_limit="23.7"/>
+      <xacro:go2_control_joint name="FL_thigh_joint" initial="0.8" effort_limit="23.7"/>
+      <xacro:go2_control_joint name="FL_calf_joint" initial="-1.5" effort_limit="35.55"/>
+      <xacro:go2_control_joint name="FR_hip_joint" effort_limit="23.7"/>
+      <xacro:go2_control_joint name="FR_thigh_joint" initial="0.8" effort_limit="23.7"/>
+      <xacro:go2_control_joint name="FR_calf_joint" initial="-1.5" effort_limit="35.55"/>
+      <xacro:go2_control_joint name="RL_hip_joint" effort_limit="23.7"/>
+      <xacro:go2_control_joint name="RL_thigh_joint" initial="0.8" effort_limit="23.7"/>
+      <xacro:go2_control_joint name="RL_calf_joint" initial="-1.5" effort_limit="35.55"/>
+      <xacro:go2_control_joint name="RR_hip_joint" effort_limit="23.7"/>
+      <xacro:go2_control_joint name="RR_thigh_joint" initial="0.8" effort_limit="23.7"/>
+      <xacro:go2_control_joint name="RR_calf_joint" initial="-1.5" effort_limit="35.55"/>
     </ros2_control>
   </xacro:macro>
