Commit message: 集成 RL policy (ONNX) + 诊断传感器问题
修改内容:
- 添加 go2_onnx_policy_node.py (50Hz RL policy 推理)
- 修改 gazebo.xacro: gpu_lidar 配置优化
- 修改 go2_sim.launch.py: 移除物理暂停机制
- 修改 run.launch.py: 集成 ONNX policy 节点
- 创建 launch_exploration_lightweight.sh: 运动学模拟器模式

已验证:
- Odometry 数据流正常 (78Hz)
- 运动学模拟器点云正常 (10Hz)
- RL policy 节点架构正确

待修复:
- Gazebo 物理模式 LiDAR 传感器无数据 (动态 spawn 时序冲突)
- 下一步: 在 SDF 中预定义 GO2 模型解决传感器问题

File: src/simulator/Utils/go2_description/xacro/gazebo.xacro (robot description, xacro)
@@ -21,15 +21,18 @@
         <parameters>$(find go2_description)/config/ros2_controllers.yaml</parameters>
       </plugin>
+      <!-- Always publish odometry, regardless of control mode -->
+      <plugin filename="ignition-gazebo-odometry-publisher-system"
+              name="gz::sim::systems::OdometryPublisher">
+        <odom_publish_frequency>100</odom_publish_frequency>
+        <dimensions>3</dimensions>
+      </plugin>
       <xacro:if value="$(arg terrain_velocity_control)">
-        <!-- Planning benchmark adapter: drives the Gazebo model from Twist
-             while physics still resolves gravity and terrain contacts. This
-             is not a learned or force-level quadruped locomotion controller. -->
+        <!-- Velocity-level base: gz subscribes to /model/go2/cmd_vel and drives
+             the model at the commanded velocity, which is what the cmd_vel-level
+             closed_loop_controller expects.  A force-based base (ApplyLinkWrench
+             plus planar_cmd_vel_adapter) has no stable operating point on this
+             robot: sliding needs more force than the stance can resist tipping. -->
         <plugin filename="ignition-gazebo-velocity-control-system"
                 name="gz::sim::systems::VelocityControl"/>
-        <plugin filename="ignition-gazebo-odometry-publisher-system"
-                name="gz::sim::systems::OdometryPublisher">
-          <odom_publish_frequency>100</odom_publish_frequency>
-          <dimensions>3</dimensions>
-        </plugin>
       </xacro:if>
     </gazebo>
@@ -42,4 +45,33 @@
       </sensor>
     </gazebo>
+    <gazebo reference="lidar_link">
+      <sensor name="exploration_lidar" type="gpu_lidar">
+        <topic>/quad_0/lidar/points</topic>
+        <update_rate>10</update_rate>
+        <lidar>
+          <scan>
+            <horizontal>
+              <samples>720</samples>
+              <resolution>1</resolution>
+              <min_angle>-3.14159265359</min_angle>
+              <max_angle>3.14159265359</max_angle>
+            </horizontal>
+            <vertical>
+              <samples>1</samples>
+              <resolution>1</resolution>
+              <min_angle>0</min_angle>
+              <max_angle>0</max_angle>
+            </vertical>
+          </scan>
+          <range>
+            <min>0.20</min>
+            <max>7.50</max>
+            <resolution>0.01</resolution>
+          </range>
+        </lidar>
+        <alwaysOn>1</alwaysOn>
+        <visualize>true</visualize>
+      </sensor>
+    </gazebo>
     <xacro:go2_foot_contact leg="FL"/>
     <xacro:go2_foot_contact leg="FR"/>

File: src/simulator/Utils/go2_description/xacro/robot.xacro (robot description, xacro)
@@ -90,4 +90,23 @@
     <link name="front_camera">
     </link>
+    <joint name="lidar_joint" type="fixed">
+        <parent link="trunk"/>
+        <child link="lidar_link"/>
+        <origin rpy="0 0 0" xyz="0.10 0 0.12"/>
+    </joint>
+    <link name="lidar_link">
+        <visual>
+            <geometry><cylinder radius="0.035" length="0.045"/></geometry>
+            <material name="lidar_dark_grey"><color rgba="0.12 0.12 0.12 1"/></material>
+        </visual>
+        <collision>
+            <geometry><cylinder radius="0.035" length="0.045"/></geometry>
+        </collision>
+        <inertial>
+            <mass value="0.05"/>
+            <inertia ixx="0.0001" ixy="0" ixz="0"
+                     iyy="0.0001" iyz="0" izz="0.0001"/>
+        </inertial>
+    </link>
     <!--
     <joint name="load_joint" type="fixed">

File: src/simulator/Utils/go2_description/xacro/ros2_control.xacro (robot description, xacro)
@@ -1,9 +1,16 @@
 <?xml version="1.0"?>
 <robot xmlns:xacro="http://www.ros.org/wiki/xacro">
-  <xacro:macro name="go2_control_joint" params="name initial:=0.0">
+  <xacro:macro name="go2_control_joint" params="name initial:=0.0 effort_limit:=33.5">
     <joint name="${name}">
       <command_interface name="position">
         <param name="min">-3.14</param>
         <param name="max">3.14</param>
+      </command_interface>
+      <!-- A locomotion policy is trained against torque-limited joint PD.  The
+           position interface cannot express that: gz_ros2_control turns a
+           position command into a velocity servo with one fixed gain. -->
+      <command_interface name="effort">
+        <param name="min">-${effort_limit}</param>
+        <param name="max">${effort_limit}</param>
       </command_interface>
       <state_interface name="position">

Commit message: Archive dyn exploration snapshot with portable Go2 launch and world resources
Preserve current Local/Explorer/Global development changes and code audit tools.
Package the current RL policy and offline NewMine assets, and add a reproducible
Fortress Campus conversion with explicit Z_UP geometry validation. Document
Humble/Fortress setup, launch commands, measured checks and known recovery and
region-display limitations.

File: src/simulator/Utils/go2_description/xacro/gazebo.xacro (robot description, xacro)
@@ -64,23 +64,23 @@
       <sensor name="exploration_lidar" type="gpu_lidar">
         <topic>/quad_0/lidar/points</topic>
-        <update_rate>10</update_rate>
+        <update_rate>${mid360.sensor.update_rate}</update_rate>
         <lidar>
           <scan>
             <horizontal>
-              <samples>720</samples>
+              <samples>${mid360.sensor.horizontal_samples}</samples>
               <resolution>1</resolution>
-              <min_angle>-3.14159265359</min_angle>
-              <max_angle>3.14159265359</max_angle>
+              <min_angle>${mid360.sensor.horizontal_min}</min_angle>
+              <max_angle>${mid360.sensor.horizontal_max}</max_angle>
             </horizontal>
             <vertical>
-              <samples>1</samples>
+              <samples>${mid360.sensor.vertical_samples}</samples>
               <resolution>1</resolution>
-              <min_angle>0</min_angle>
-              <max_angle>0</max_angle>
+              <min_angle>${mid360.sensor.vertical_min}</min_angle>
+              <max_angle>${mid360.sensor.vertical_max}</max_angle>
             </vertical>
           </scan>
           <range>
-            <min>0.20</min>
-            <max>7.50</max>
+            <min>${mid360.sensor.range_min}</min>
+            <max>${mid360.sensor.range_max}</max>
             <resolution>0.01</resolution>
           </range>

File: src/simulator/Utils/go2_description/xacro/robot.xacro (robot description, xacro)
@@ -1,4 +1,5 @@
 <?xml version="1.0"?>
 <robot name="go2" xmlns:xacro="http://www.ros.org/wiki/xacro">
+    <xacro:property name="mid360" value="${xacro.load_yaml('$(find go2_description)/config/mid360.yaml')}"/>
     <xacro:arg name="DEBUG" default="false"/>
     <xacro:arg name="use_gazebo" default="true"/>
@@ -98,5 +99,8 @@
         <parent link="trunk"/>
         <child link="lidar_link"/>
-        <origin rpy="0 0 0" xyz="0.10 0 0.12"/>
+        <!-- Unitree kit is pitched down 13deg. Keep TF and both mappers
+             on the same profile; sensor-local elevation remains -7..52deg. -->
+        <origin rpy="${mid360.mount.roll} ${mid360.mount.pitch} ${mid360.mount.yaw}"
+                xyz="${mid360.mount.x} ${mid360.mount.y} ${mid360.mount.z}"/>
     </joint>
     <link name="lidar_link">
